File: ErgoMaxRight/ErgoMaxRight.kicad_sch (KiCad schematic)
At the start: 103 parts, among them J1 PJ-320A, K1 F12, K10 8 *, K11 7 &, K12 6 ^, K13 KEYSW, K14 KEYSW, K15 P, K16 O, K17 I, K18 U, K19 Y, K2 F11, K20 KEYSW, K21 KEYSW, K22 ; :, K23 L, K24 K, K25 J, K26 H, K27 KEYSW, K28 KEYSW, K29 KEYSW, K3 F10, K30 / ?, K31 . >, K32 , <, K33 M, K34 N, K35 KEYSW, K36 KEYSW, K37 KEYSW, K38 KEYSW, K39 KEYSW, K4 F9, K40 KEYSW, K41 KEYSW, K42 KEYSW, K43 KEYSW, K44 KEYSW, K5 F8, K6 F7, K7 KEYSW, K8 0 ), K9 9 (, U1 ProMicro

Commit message: updated for jlcpcb available components
Parts:
- J1: LCSC C2884926 -> (none)
- K1, K10, K11, K12, K15, K16, K17, K18, K19, K2, K22, K23, K24, K25, K26, K3, K30, K31, K32, K33, K34, K4, K5, K6, K8, K9: LCSC C2803348 -> C5184526
- K13: value KEYSW -> K13; LCSC C2803348 -> C5184526
- K14: value KEYSW -> K14; LCSC C2803348 -> C5184526
- K20: value KEYSW -> K20; LCSC C2803348 -> C5184526
- K21: value KEYSW -> K21; LCSC C2803348 -> C5184526
- K27: value KEYSW -> K27; LCSC C2803348 -> C5184526
- K28: value KEYSW -> K28; LCSC C2803348 -> C5184526
- K29: value KEYSW -> K29; LCSC C2803348 -> C5184526
- K35: value KEYSW -> K35; LCSC C2803348 -> C5184526
- K36: value KEYSW -> K36; LCSC C2803348 -> C5184526
- K37: value KEYSW -> K37; LCSC C2803348 -> C5184526
- K38: value KEYSW -> K38; LCSC C2803348 -> C5184526
- K39: value KEYSW -> K39; LCSC C2803348 -> C5184526
- K40: value KEYSW -> K40; LCSC C2803348 -> C5184526
- K41: value KEYSW -> K41; LCSC C2803348 -> C5184526
- K42: value KEYSW -> K42; LCSC C2803348 -> C5184526
- K43: value KEYSW -> K43; LCSC C2803348 -> C5184526
- K44: value KEYSW -> K44; LCSC C2803348 -> C5184526
- K7: value KEYSW -> K7; LCSC C2803348 -> C5184526
- R1, R2: LCSC C4241436 -> C352105
